File: lm3409.sch (KiCad schematic (older format))
At the start: 19 parts, among them Q1 NTD20P06LT4G, U1 LM3409HV

Commit message: Update values
Parts:
- R2: value DNF -> 178K
- R3: value TBD -> 16K2
- R4: value TBD -> 6K98
- R5: value TBD -> 49K9
Changed lines of the file:
@@
 P 5000 2750
 F 0 "R5" V 4703 2750 50  0000 C CNN
-F 1 "TBD" V 4794 2750 50  0000 C CNN
+F 1 "49K9" V 4794 2750 50  0000 C CNN
 F 2 "Resistor_SMD:R_0603_1608Metric" V 4885 2750 50  0000 C CNN
 F 3 "~" H 5000 2750 50  0001 C CNN
@@
 P 4125 3300
 F 0 "R4" V 3828 3300 50  0000 C CNN
-F 1 "TBD" V 3919 3300 50  0000 C CNN
+F 1 "6K98" V 3919 3300 50  0000 C CNN
 F 2 "Resistor_SMD:R_0603_1608Metric" V 4000 2875 50  0000 C CNN
 F 3 "~" H 4125 3300 50  0001 C CNN
@@
 P 3750 3600
 F 0 "R3" V 3750 3075 50  0000 C CNN
-F 1 "TBD" V 3825 3075 50  0000 C CNN
+F 1 "16K2" V 3825 3075 50  0000 C CNN
 F 2 "Resistor_SMD:R_0603_1608Metric" V 3925 3075 50  0000 C CNN
 F 3 "~" H 3750 3600 50  0001 C CNN
@@
 P 2675 3400
 F 0 "R2" V 2378 3400 50  0000 C CNN
-F 1 "DNF" V 2469 3400 50  0000 C CNN
+F 1 "178K" V 2469 3400 50  0000 C CNN
 F 2 "Resistor_SMD:R_0603_1608Metric" V 2550 2975 50  0000 C CNN
 F 3 "~" H 2675 3400 50  0001 C CNN
