File: lm3409.kicad_pcb (KiCad board)
At the start: 2 copper layers, 29.2 x 37.5 mm, 22 parts, among them Q1 NTD20P06LT4G, U1 LM3409HV

Commit message: Update values
Parts:
- R4: value TBD -> 6K98
- R5: value TBD -> 49K9

Commit message: Update lm3409.kicad_pcb
Parts:
- R2: value DNF -> 178K
